File: hardware/MainBoard/MainBoard.kicad_pcb (KiCad board)
At the start: 2 copper layers, 45 x 80 mm, 29 parts, among them J1 to front board, J2 to front board, J5 Bus 1 power/MIDI, J6 Bus 2 audio, J7 DEBUG UART0, U1 H11L1

Commit message: Give BOOT a spring pin so the module stays a plug-in part
BOOT was the only signal on either board that did not end on a connector
pin: it stopped at TP1, a solder pad, and a hand-soldered wire finished
the job at the module's underside. That works, but the sockets are in the
BOM specifically to keep the module replaceable, and a wire tethers it.

TP2 is a landing pad at 26.51 / 7.58, under the module's BOOT pad, for a
spring-loaded pin spanning 11.04 mm -- socket body 8.5 plus header plastic
2.54, both read out of their own STEP models. Seating the module makes the
contact. TP1 stays, out at the edge where an iron reaches, because two
things about that position are unsettled: the coordinate comes from the
Raspberry Pi Pico 2 datasheet and the module is a WeAct RP2350-Plus with
its own layout, and the sign of X depends on which side that drawing is
viewed from. Both are settled by looking at the part -- is the pad nearer
the GP0 row or the VBUS row -- and only that one number changes. If it
turns out to be somewhere else entirely, it is the short-wire build after
all and nothing is lost.

The pad landed on UART0_RX, so that net was laid again. The first attempt
then took the corridor past C9 and pinched the ground pour into an 8.4 mm²
island with C9's own ground pad inside it -- the RUN capacitor would have
had no return path. Too narrow for a stitching via (widest point 0.468 mm,
a 0.6 mm via needs 0.50), so the corridor is a router keep-out now and
UART0_RX goes round.

Both boards: 0 open DRC, 0 unconnected, 0 parity, ERC 0 on all three
schematics. One documented exclusion, for TP2's hole sitting inside A1's
courtyard -- that pair only, so the rule still guards the rest of the
board.

Co-Authored-By: Claude Opus 5 <noreply@anthropic.com>
Parts:
- added TP2: BOOT pogo, TestPoint:TestPoint_THTPad_D2.0mm_Drill1.0mm, B.Cu at (26.5, 7.58)
Routing:
- net BOOT: track 17.1 -> 72.2 mm, vias 0 -> 2
- net /Main board/UART0_RX: track 53.6 -> 59.0 mm
- net GND: vias 11 -> 12

Commit message: TP6 is at (8, 38), not where I had it
Michael's photo said the test point looked wrong, and it was: 7.7 mm
wrong. The pad moves from 26.51 / 7.58 to 25.00 / 15.13.

Both coordinate sets I had been given were second-hand and neither
matched. Figure 5 of the Pico 2 datasheet settles it -- the SMT footprint,
test-point centres in a frame whose origin is the board's bottom-left
corner, USB shell pads at x 7.775 and 13.225 fixing the centreline at
10.5. The frame checks out independently: it puts pin 1's centre 1.37 mm
from the top edge, exactly what KiCad's Pico footprint uses.

The drawing gives seven test points and labels none of them, so which one
is TP6 had to be reasoned out. Three sit at the USB connector -- TP1 to
TP3, the USB group. Of the column at x = 8, the one at y = 43 is 8.0 mm
from that end and the LED is at 7.4; the one at y = 38 is 13.0 mm and the
BOOTSEL button is at 13.2. Both measured off a photo of the board, and
they leave one reading. (11.5, 30.5) is TP7 over by the chip.

Two things get easier: the pad is 1.5 x 1.5 mm rather than the 1 mm round
I had been working to, and BOOT comes out 67.2 mm instead of 72.2. The
silk trim on A1's USB outline is reverted -- that was to clear the old
position and is not needed at the new one.

Both boards: 0 open DRC, 0 unconnected, 0 parity.

Co-Authored-By: Claude Opus 5 <noreply@anthropic.com>
Parts:
- moved TP2 7.70 mm to (25.0, 15.1)
Routing:
- net BOOT: track 72.2 -> 67.2 mm
Changed lines of the file:
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@@
 	(footprint "TestPoint:TestPoint_THTPad_D2.0mm_Drill1.0mm"
 		(layer "B.Cu")
-		(at 26.51 7.58)
+		(at 25 15.13)
 		(descr "THT pad as test Point, diameter 2.0mm, hole diameter 1.0mm")
 		(property "Reference" "TP2"
@@
 			(net "BOOT")
 		)
+		(embedded_fonts no)
 		(model "${KIPRJMOD}/../3dmodels/SpringPin_11mm_Stand-in.wrl"
-			(offset (xyz 0 0 0))
-			(scale (xyz 1 1 1))
-			(rotate (xyz 0 0 0))
+			(offset
+				(xyz 0 0 0)
+			)
+			(scale
+				(xyz 1 1 1)
+			)
+			(rotate
+				(xyz 0 0 0)
+			)
 		)
-		(embedded_fonts no)
 	)
 	(footprint "Connector_PinHeader_2.54mm:PinHeader_1x03_P2.54mm_Vertical"
@@
 		(fp_line
 			(start 12.79 -3.04)
-			(end 5.9 -3.04)
+			(end 4.99 -3.04)
 			(stroke
 				(width 0.12)
@@
 		)
 		(fp_line
-			(start 5.9 -1.824)
-			(end 5.9 -3.04)
+			(start 5.29 -49.74)
+			(end 3.652061 -49.74)
 			(stroke
 				(width 0.12)
@@
 		)
 		(fp_line
-			(start 5.29 -49.74)
-			(end 3.652061 -49.74)
+			(start 4.99 1.96)
+			(end 4.99 0.564)
 			(stroke
 				(width 0.12)
@@
 		)
 		(fp_line
-			(start 4.99 1.96)
-			(end 4.99 0.564)
+			(start 4.99 -1.824)
+			(end 4.99 -3.04)
 			(stroke
 				(width 0.12)
@@
 	)
 	(segment
-		(start 14.859 19.304)
-		(end 16.383 17.78)
-		(width 0.2)
-		(layer "F.Cu")
-		(net "BOOT")
-	)
-	(segment
-		(start 12.573 20.066)
-		(end 14.605 20.066)
+		(start 7.112 31.242)
+		(end 7.112 31.115)
 		(width 0.2)
 		(layer "F.Cu")
@@
 	)
 	(segment
-		(start 7.239 25.4)
-		(end 12.573 20.066)
+		(start 6.096 34.798)
+		(end 6.477 34.417)
 		(width 0.2)
 		(layer "F.Cu")
@@
 	)
 	(segment
-		(start 6.096 34.798)
-		(end 6.477 34.417)
-		(width 0.2)
-		(layer "F.Cu")
-		(net "BOOT")
-	)
-	(segment
-		(start 14.605 20.066)
-		(end 14.732 19.939)
+		(start 7.239 25.4)
+		(end 12.573 20.066)
 		(width 0.2)
 		(layer "F.Cu")
@@
 	)
 	(segment
-		(start 7.112 31.242)
-		(end 7.112 31.115)
-		(width 0.2)
-		(layer "F.Cu")
-		(net "BOOT")
-	)
-	(segment
-		(start 14.732 19.939)
-		(end 14.732 19.812)
-		(width 0.2)
-		(layer "F.Cu")
-		(net "BOOT")
-	)
-	(segment
-		(start 14.859 19.685)
-		(end 14.859 19.304)
-		(width 0.2)
-		(layer "F.Cu")
-		(net "BOOT")
-	)
-	(segment
-		(start 14.732 19.812)
-		(end 14.859 19.685)
+		(start 12.573 20.066)
+		(end 18.542 20.066)
 		(width 0.2)
 		(layer "F.Cu")
@@
 	)
 	(via
-		(at 16.383 17.78)
+		(at 18.542 20.066)
 		(size 0.6)
 		(drill 0.3)
@@
 	)
 	(segment
-		(start 5 52.5)
-		(end 4.953 35.941)
+		(start 6.096 53.848)
+		(end 5.969 53.721)
 		(width 0.2)
 		(layer "B.Cu")
@@
 	)
 	(segment
-		(start 5.969 53.721)
-		(end 5.969 53.467)
+		(start 20.066 20.066)
+		(end 25 15.13)
 		(width 0.2)
 		(layer "B.Cu")
@@
 	)
 	(segment
-		(start 7.747 56.515)
-		(end 7.62 56.515)
+		(start 18.923 55.372)
+		(end 17.653 56.642)
 		(width 0.2)
 		(layer "B.Cu")
@@
 	)
 	(segment
-		(start 4.953 35.941)
-		(end 6.096 34.798)
+		(start 19.05 55.4)
+		(end 18.923 55.372)
 		(width 0.2)
 		(layer "B.Cu")
@@
 	)
 	(segment
-		(start 16.383 17.78)
-		(end 26.51 7.58)
+		(start 7.62 55.499)
+		(end 6.096 53.975)
 		(width 0.2)
 		(layer "B.Cu")
@@
 	)
 	(segment
-		(start 18.923 55.372)
-		(end 17.653 56.642)
+		(start 5 52.5)
+		(end 4.953 35.941)
 		(width 0.2)
 		(layer "B.Cu")
@@
 	)
 	(segment
-		(start 17.653 56.642)
-		(end 7.747 56.642)
+		(start 7.747 56.642)
+		(end 7.747 56.515)
 		(width 0.2)
 		(layer "B.Cu")
@@
 	)
 	(segment
-		(start 19.05 55.4)
-		(end 18.923 55.372)
+		(start 4.953 35.941)
+		(end 6.096 34.798)
 		(width 0.2)
 		(layer "B.Cu")
@@
 	)
 	(segment
-		(start 7.747 56.642)
-		(end 7.747 56.515)
+		(start 18.542 20.066)
+		(end 20.066 20.066)
+		(width 0.2)
+		(layer "B.Cu")
+		(net "BOOT")
+	)
+	(segment
+		(start 17.653 56.642)
+		(end 7.747 56.642)
 		(width 0.2)
 		(layer "B.Cu")
@@
 	)
 	(segment
-		(start 7.62 55.499)
-		(end 6.096 53.975)
+		(start 7.747 56.515)
+		(end 7.62 56.515)
 		(width 0.2)
 		(layer "B.Cu")
@@
 	)
 	(segment
-		(start 6.096 53.975)
-		(end 6.096 53.848)
+		(start 5.969 53.467)
+		(end 5 52.5)
 		(width 0.2)
 		(layer "B.Cu")
@@
 	)
 	(segment
-		(start 6.096 53.848)
-		(end 5.969 53.721)
+		(start 5.969 53.721)
+		(end 5.969 53.467)
 		(width 0.2)
 		(layer "B.Cu")
@@
 	)
 	(segment
-		(start 5.969 53.467)
-		(end 5 52.5)
+		(start 6.096 53.975)
+		(end 6.096 53.848)
 		(width 0.2)
 		(layer "B.Cu")
